Commit message: Setup home configuration

File: my_robot/robot.urdf (robot description, URDF)
Before this commit: robot LAB0_urdf, 4 links, 3 joints
Joints:
- joint joint_B2L1: origin xyz=0.00888631783719275 -0.184033872630811 0.0532600398559306 rpy=1.5707963267949 0 -0.347221884464147 -> xyz=0 0 0 rpy=1.5707963267949 0 1.5707963267949

Commit message: add effector

File: my_robot/robot.urdf (robot description, URDF)
Before this commit: robot LAB0_urdf, 4 links, 3 joints
Links:
- added link end_effector
Joints:
- added joint end_effector_joint: type fixed, parent Prismatic_link, child end_effector, origin xyz=0 0 0 rpy=0 0 0

Commit message: git push la

File: my_robot/robot.urdf (robot description, URDF)
Before this commit: robot LAB0_urdf, 5 links, 4 joints
Links:
- removed link LInk2
- removed link Link1
- removed link Prismatic_link
- removed link end_effector
- added link ee_link, mass 16.5300550651784
- added link joint_1_link, mass 2.74003858179814; collision mesh filename=package://my_robot/meshes/joint_1_link.STL; visual mesh filename=package://my_robot/meshes/joint_1_link.STL
- added link joint_2_link, mass 9.82047843595601; collision mesh filename=package://my_robot/meshes/joint_2_link.STL; visual mesh filename=package://my_robot/meshes/joint_2_link.STL
- added link joint_3_link, mass 2.6; collision mesh filename=package://my_robot/meshes/joint_3_link.STL; visual mesh filename=package://my_robot/meshes/joint_3_link.STL
Joints:
- removed joint Prsimatic_joint
- removed joint end_effector_joint
- removed joint joint_B2L1
- removed joint joint_L12L2
- added joint ee_joint: type fixed, parent joint_3_link, child ee_link, origin xyz=0 0 0.4 rpy=0 0 0, axis 0 0 0
- added joint joint_1_joint: type revolute, parent base_link, child joint_1_link, origin xyz=0 0 0 rpy=0 0 0, axis 0 0 1, limit lower=0 upper=0 effort=0 velocity=0
- added joint joint_2_joint: type revolute, parent joint_1_link, child joint_2_link, origin xyz=0 0 0.51 rpy=1.5708 0 0, axis 0 0 1, limit lower=0 upper=0 effort=0 velocity=0
- added joint joint_3_joint: type prismatic, parent joint_2_link, child joint_3_link, origin xyz=0.1 0 0 rpy=1.5708 0 1.5708, axis 0 0 -1, limit lower=0 upper=0 effort=0 velocity=0
